File: HelloBoard.kicad_pcb (KiCad board)
At the start: 2 copper layers, 106.3 x 77 mm, 43 parts, among them J1 USB_B_Micro, J2 Conn_01x04_Pin, J3 Conn_01x04_Pin, J4 Conn_02x08_Top_Bottom, J5 Conn_01x02, SW1 SW_Push, SW2 SW_Push, U1 STM32F103C8T6, U2 AMS1117-3.3, U3 TMP235A2DCKR, U4 ADXL343, Y1 16MHz

Commit message: gonna try stuff, checkpoint
Parts:
- added R10: 220, Resistor_SMD:R_0402_1005Metric, F.Cu at (190.3, 58.9)
- added R11: 220, Resistor_SMD:R_0402_1005Metric, F.Cu at (190.3, 56.3)
- added R12: 220, Resistor_SMD:R_0402_1005Metric, F.Cu at (190.3, 54.9)
- added R13: 220, Resistor_SMD:R_0402_1005Metric, F.Cu at (190.0, 69.4)
- added R14: 220, Resistor_SMD:R_0402_1005Metric, F.Cu at (190.1, 64.6)
- added R15: 220, Resistor_SMD:R_0402_1005Metric, F.Cu at (190.1, 66.2)
- added R16: 220, Resistor_SMD:R_0402_1005Metric, F.Cu at (190.0, 67.9)
- added R8: 220, Resistor_SMD:R_0402_1005Metric, F.Cu at (190.2, 63.2)
- added R9: 220, Resistor_SMD:R_0402_1005Metric, F.Cu at (190.3, 57.6)
- moved LED1 9.91 mm to (205.2, 62.5)
Connections:
- LED1 pad 1: /7SEG_C -> /C
- LED1 pad 10: /7SEG_A -> /A
- LED1 pad 3: /7SEG_E -> /E
- LED1 pad 4: /7SEG_D -> /D
- LED1 pad 5: /7SEG_G -> /G
- LED1 pad 6: /7SEG_F -> /F
- LED1 pad 7: /7SEG_D2_CA -> /D2_CA
- LED1 pad 8: /7SEG_D1_CA -> /D1_CA
- LED1 pad 9: /7SEG_B -> /B
Routing:
- net +3.3V: track 35.8 -> 266.7 mm, vias 0 -> 6
- net VBUS: track 87.9 -> 219.9 mm, vias 0 -> 2
- net /PA_7: track 3.33 -> 123.4 mm, vias 0 -> 4
- net /PB_2: track 3.22 -> 120.7 mm
- net /PB_1: track 3.23 -> 119.3 mm
- net /PA_12: track 0.00 -> 46.9 mm, vias 0 -> 4
- net /PA_11: track 0.00 -> 46.1 mm, vias 0 -> 4
- net /USER_BUTTON: track 6.74 -> 49.8 mm, vias 0 -> 4
- net /PA_8: track 0.00 -> 42.7 mm, vias 0 -> 4
- net /7SEG_B: track 0.00 -> 35.6 mm, vias 0 -> 2
- net /7SEG_D2_CA: track 0.00 -> 34.3 mm, vias 0 -> 2
- net /7SEG_A: track 0.00 -> 34.0 mm, vias 0 -> 3
- net /7SEG_D1_CA: track 0.00 -> 27.5 mm
- net /7SEG_D: track 4.29 -> 31.2 mm, vias 0 -> 2
- net /7SEG_G: track 0.00 -> 26.8 mm, vias 0 -> 2
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- added copper zone on F.Cu, net +3.3V
- added copper zone on F.Cu, net GND
- added copper zone on F.Cu, net VBUS
