File: HelloBoard.kicad_pcb (KiCad board)
At the start: 2 copper layers, 106.3 x 77 mm, 56 parts, among them J1 USB_B_Micro, J2 Conn_01x04_Pin, J3 Conn_01x04_Pin, J4 Conn_02x08_Top_Bottom, J5 Conn_01x02, Q1 AO3401A, Q2 AO3401A, SW1 SW_Push, SW2 SW_Push, U1 STM32F103C8T6, U2 AMS1117-3.3, U3 TMP235A2DCKR, U4 ADXL343, Y1 16MHz

Commit message: BOM preparation
Routing:
- net VBUS: track 243.6 -> 197.4 mm, vias 1 -> 0
- net +3.3V: track 336.4 -> 329.6 mm, vias 9 -> 14
- net /D2_CA: track 31.3 -> 29.8 mm
- net /PA_9: track 52.5 -> 51.6 mm
- net GND: track 56.0 -> 56.9 mm
- net /USER_BUTTON: track 71.4 -> 70.6 mm
- net /LCD_VO: track 26.5 -> 27.2 mm, vias 0 -> 1
- net /PA_10: track 49.3 -> 48.7 mm

Commit message: backside silkscreen added
Parts:
- added G***: LOGO, SilkScreen:bee, B.Cu at (162.9, 95.4)
- added G***: LOGO, SilkScreen:rocky, B.Cu at (143.1, 97.6)
- added G***: LOGO, SilkScreen:theo, B.Cu at (183.8, 107.1)
- added G***: LOGO, SilkScreen:bob, B.Cu at (137.4, 108.3)
- added G***: LOGO, SilkScreen:steve, B.Cu at (185.7, 96.5)
- added G***: LOGO, SilkScreen:puck, B.Cu at (165.5, 109.4)
- added G***: LOGO, SilkScreen:omarqm, B.Cu at (194.6, 95.5)
- added G***: LOGO, SilkScreen:potatoblood, B.Cu at (157.3, 109.8)
- added G***: LOGO, SilkScreen:kirby, B.Cu at (203.8, 101.0)
- added G***: LOGO, SilkScreen:anakin, B.Cu at (213.8, 101.8)
- added G***: LOGO, SilkScreen:asha, B.Cu at (173.8, 104.5)
- added G***: LOGO, SilkScreen:kuriboh, B.Cu at (188.9, 84.0)
- added G***: LOGO, SilkScreen:mnrn, B.Cu at (148.9, 109.2)
- added G***: LOGO, SilkScreen:marwan, B.Cu at (135.9, 98.3)
- added G***: LOGO, SilkScreen:usagi, B.Cu at (174.8, 95.7)
- added G***: LOGO, SilkScreen:turtle, B.Cu at (194.0, 107.4)

Commit message: more backside silkscreen
Parts:
- added G***: LOGO, SilkScreen:pickle, B.Cu at (152.8, 96.3)

Commit message: .
Parts:
- added G***: LOGO, SilkScreen:finn, B.Cu at (182.8, 85.2)
- moved G*** 8.94 mm to (197.8, 84.8)
